Commit message: Add whole uv body and cameras

File: src/Final_Project/vtec_u3_description/urdf/base.xacro (robot description, xacro)
@@ -39,13 +39,12 @@
                    izz="0.64879823" /> -->
           <!-- For COM nearly in geometric center -->
-            <!-- inertia ixx="0.83639798529" ixy="-0.00503680373" ixz="0.0560001532"
+            <inertia ixx="0.83639798529" ixy="-0.00503680373" ixz="0.0560001532"
                       iyy="0.46118483068" iyz="-0.01377965358"
-                      izz="1.02986207702" /-->
+                      izz="1.02986207702" />
         </inertial>
         <visual>
           <origin xyz="${geocenter}" rpy="0 0 0"/>
           <geometry>
-            <box size= "0.6 0.6 0.6"/>
-            <!-- mesh filename="${visual_mesh_file}" scale="0.001 0.001 0.001" /-->
+            <mesh filename="${visual_mesh_file}" scale="0.001 0.001 0.001" />
           </geometry>
         </visual>

File: src/Final_Project/vtec_u3_description/urdf/sensors.xacro (robot description, xacro)
@@ -35,8 +35,8 @@
     <origin xyz="0.19281 0.01961 0.06659" rpy="0 0 0"/>
   </xacro:realsense_camera>
-  <!-- Realsense R200 - ->
+  <!-- Realsense R200 -->
   <xacro:realsense_camera namespace="${namespace}" parent_link="${namespace}/base_link" suffix="down">
     <origin xyz="2.19281 0.01961 0.06659" rpy="0 1.57 0"/>
-  </xacro:realsense_camera-->
+  </xacro:realsense_camera>
   <!-- Realsense R200 -->
   <!-- Import macro for realsense-RS200 camera-->
