Commit message: .

File: src/Final_Project/sim_challenges/urdf/bin1.xacro (robot description, xacro)
@@ -6,5 +6,5 @@
 <link name="bin1_base">
     <visual>
-        <origin xyz="5.00 0 -22.0" rpy="0.0 0.0 -1.57"/>
+        <origin xyz="10 0 0" rpy="0.0 0.0 -1.57"/>
         <geometry>
             <mesh filename="${visual_mesh_file}" scale="1 1 1" />
@@ -13,5 +13,5 @@
         <!-- Se deben cambiar los parametros reales-->
     <collision>
-      <origin xyz="5.00 0 -22.0" rpy="0.0 0.0 -1.57"/>
+      <origin xyz="10 0 0" rpy="0.0 0.0 -1.57"/>
       <geometry>
         <mesh filename="${visual_mesh_file}" scale="1 1 1" />
@@ -19,5 +19,5 @@
     </collision>
     <inertial>
-      <origin xyz="5.00 0 -22.0" rpy="0.0 0.0 -1.57"/>
+      <origin xyz="10 0 0" rpy="0.0 0.0 -1.57"/>
       <mass value="1"/>
       <inertia

File: src/Final_Project/sim_challenges/urdf/bin2.xacro (robot description, xacro)
@@ -6,5 +6,5 @@
 <link name="bin2_base">
     <visual>
-        <origin xyz="5.00 0 -22.0" rpy="0.0 0.0 -1.57"/>
+        <origin xyz="10 0 0" rpy="0.0 0.0 -1.57"/>
         <geometry>
             <mesh filename="${visual_mesh_file}" scale="1 1 1" />
@@ -13,5 +13,5 @@
         <!-- Se deben cambiar los parametros reales-->
     <collision>
-      <origin xyz="5.00 0 -22.0" rpy="0.0 0.0 -1.57"/>
+      <origin xyz="10 0 0" rpy="0.0 0.0 -1.57"/>
       <geometry>
         <mesh filename="${visual_mesh_file}" scale="1 1 1" />
@@ -19,5 +19,5 @@
     </collision>
     <inertial>
-      <origin xyz="5.00 0 -22.0" rpy="0.0 0.0 -1.57"/>
+      <origin xyz="10 0 0" rpy="0.0 0.0 -1.57"/>
       <mass value="1"/>
       <inertia

Commit message: bin1.xacro modified

File: src/Final_Project/sim_challenges/urdf/bin1.xacro (robot description, xacro)
@@ -1,7 +1,7 @@
 <?xml version="1.0"?>
+<!-- Con este archivo.xacro te puedes guiar para hacer los otros, si tienes duda
+de lo que se debe cambiar sigue la presentacion <<Proyecto Final>>> -->
 <robot name="bin_1" xmlns:xacro="http://www.ros.org/wiki/xacro">
-<!-- Introducir meshes -->
 <xacro:property name="visual_mesh_file" value="file://$(find sim_challenges)/models/meshes/bin.dae" />
-<!-- <origin xyz="0.085 (0 -0.085) 0 0" rpy="0.0 0.0 1.57075"/> -->
 <link name="bin1_base">
     <visual>
@@ -11,5 +11,4 @@
         </geometry>
     </visual>
-        <!-- Se deben cambiar los parametros reales-->
     <collision>
       <origin xyz="10 0 0" rpy="0.0 0.0 -1.57"/>
